File: hardware/proto-0/baseboard/accelerator-devkit-proto-0-baseboard-display-io.kicad_sch (KiCad schematic)
At the start: 17 parts, among them J7 Display, U1 LFE5U-45-caBGA256, U14 TPS61046YFFR

Commit message: Moving all power rail test points to the front
Parts:
- TP2: footprint TestPoint:TestPoint_Pad_D1.0mm -> TestPoint:TestPoint_THTPad_D1.0mm_Drill0.5mm
Changed lines of the file:
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@@
 (kicad_sch (version 20200512) (host eeschema "(5.99.0-1839-gb83d64fc0)")
-  (page 1 8)
+  (page 8 8)
   (paper "USLetter")
   (title_block
@@
   (no_connect (at 168.91 40.64))
   (no_connect (at 168.91 63.5))
+  (no_connect (at 168.91 53.34))
+  (no_connect (at 168.91 43.18))
+  (no_connect (at 168.91 48.26))
   (no_connect (at 168.91 50.8))
-  (no_connect (at 168.91 48.26))
-  (no_connect (at 168.91 43.18))
-  (no_connect (at 168.91 53.34))
   (wire (pts (xy 17.78 57.15) (xy 40.64 57.15))
     (stroke (width 0) (type solid) (color 0 0 0 0))
@@
       (effects (font (size 1.27 1.27)) (justify left) hide)
     )
-    (property "Footprint" "TestPoint:TestPoint_Pad_D1.0mm" (id 2) (at 191.77 135.89 0)
+    (property "Footprint" "TestPoint:TestPoint_THTPad_D1.0mm_Drill0.5mm" (id 2) (at 191.77 135.89 0)
       (effects (font (size 1.27 1.27)) hide)
     )
