File: hardware/proto-0/baseboard/accelerator-devkit-proto-0-baseboard-fpga-io.kicad_sch (KiCad schematic)
At the start: 24 parts, among them J4 Qwiic I2C, J5 Pmod 1A, J6 Pmod 1B, J8 microSD-ST11-H, SW1 BUTTON1, SW2 BUTTON2, SW3 BUTTON3, SW4 SWITCH, U1 LFE5U-45-caBGA256, U13 TPD4E05U06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

Commit message: Removing unused MP Pin on Qwiic connector
Parts:
- J4: symbol Connector_Generic_MountingPin:Conn_01x04_MountingPin -> Connector_Generic:Conn_01x04
Connections:
- no-connect marks 11 -> 10
Changed lines of the file:
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@@
 (kicad_sch (version 20200512) (host eeschema "(5.99.0-1839-gb83d64fc0)")
-  (page 1 8)
+  (page 6 8)
   (paper "USLetter")
   (title_block
@@
   (junction (at 203.2 105.41))
   (junction (at 203.2 119.38))
+  (no_connect (at 142.24 17.78))
+  (no_connect (at 173.99 115.57))
   (no_connect (at 173.99 123.19))
+  (no_connect (at 113.03 161.29))
   (no_connect (at 173.99 118.11))
   (no_connect (at 173.99 110.49))
-  (no_connect (at 142.24 17.78))
-  (no_connect (at 102.87 16.51))
-  (no_connect (at 172.72 161.29))
-  (no_connect (at 113.03 161.29))
-  (no_connect (at 173.99 115.57))
-  (no_connect (at 106.68 179.07))
   (no_connect (at 142.24 22.86))
   (no_connect (at 106.68 173.99))
+  (no_connect (at 172.72 161.29))
+  (no_connect (at 106.68 179.07))
   (wire (pts (xy 19.05 22.86) (xy 40.64 22.86))
     (stroke (width 0) (type solid) (color 0 0 0 0))
@@
     )
   )
-  (symbol (lib_id "Connector_Generic_MountingPin:Conn_01x04_MountingPin") (at 102.87 26.67 0) (mirror x) (unit 1)
+  (symbol (lib_id "Connector_Generic:Conn_01x04") (at 102.87 26.67 0) (mirror x) (unit 1)
     (property "Reference" "J4" (id 0) (at 105.004 24.517 0)
       (effects (font (size 1.27 1.27)) (justify left))
